File: StringLightsController.kicad_pcb (KiCad board)
At the start: 2 copper layers, 48 x 57 mm, 59 parts, among them J1 5V_IN, J2 RF_RX, J3 SERIAL+GPIO, J4 LAMPS_A, J5 LAMPS_B, Q1 IRF7319TRPBF, Q2 IRF7319TRPBF, Q3 IRF7319TRPBF, Q4 IRF7319TRPBF, SW1 RESET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

Commit message: Add BoM
Parts:
- R17, R18, R19, R20: value 5K6 -> 4K7
