File: StringLightsController.kicad_sch (KiCad schematic)
At the start: 59 parts, among them J1 5V_IN, J2 RF_RX, J3 SERIAL+GPIO, J4 LAMPS_A, J5 LAMPS_B, Q1 IRF7319TRPBF, Q2 IRF7319TRPBF, Q3 IRF7319TRPBF, Q4 IRF7319TRPBF, SW1 RESET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

Commit message: Add BoM
Parts:
- C1, C6: MPN1 (none) -> UWR1A101MCL1GB; Part UWR1A101MCL1GB -> (none)
- C10, C9: MPN1 (none) -> UWT1A102MNL1GS; Part UWT1A102MNL1GS -> (none)
- C13, C14, C7: MPN1 (none) -> CC0805KRX7R7BB104; Part CC0805KRX7R7BB104 -> (none)
- C2: MPN1 (none) -> AFK106M25B12T-F; Part AFK106M25B12T-F -> (none)
- D4, D5: MPN1 (none) -> SS34FA
- JP1: MPN1 N/A -> (none)
- Q1, Q2, Q3, Q4: MPN1 (none) -> IRF7319TRPBF
- R10, R11, R12, R13, R14, R15, R16, R9: MPN1 (none) -> RC0805FR-07100RL
- R17, R18, R19, R20: value 5K6 -> 4K7; MPN1 (none) -> RC0805FR-074K7L
- U1: MPN1 ESP32-WROOM-32D -> ESP32-WROOM-32D-N4
- U2: MPN1 (none) -> AP2112K-3.3
- U3, U4: MPN1 (none) -> AP2112K-2.5
